File: Split Keyboard.kicad_sch (KiCad schematic)
At the start: 2 parts, among them J1 USB_C_Receptacle_USB2.0_16P

Commit message: Created the PCB layout
Parts:
- J1: footprint (none) -> Connector_USB:USB_C_Receptacle_XKB_U262-16XN-4BVC11
Changed lines of the file:
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@@
 			)
 		)
-		(property "Footprint" ""
+		(property "Footprint" "Connector_USB:USB_C_Receptacle_XKB_U262-16XN-4BVC11"
 			(at 269.24 162.56 0)
 			(hide yes)
